File: _saved_little_mobile_stm32f0.sch (KiCad schematic (older format))
At the start: 5 parts, among them J1 USB_OTG, J2 BAT+ Contact, J3 BAT- Contact, J4 Header_SWD

Commit message: pcb Layout nearly completed
Parts:
- J1: footprint (none) -> little_mobile_stm32f0:Molex_1050170001_MicroUSB_B
- J2, J3: footprint (none) -> little_mobile_stm32f0:KEYSTONE_109-2_Battery_Contact
- J4: footprint Pin_Headers:Pin_Header_Angled_1x03_Pitch2.54mm -> Pin_Headers:Pin_Header_Straight_1x03_Pitch2.54mm
Changed lines of the file:
@@
 F 0 "J2" H 2300 1450 50  0000 C CNN
 F 1 "BAT+ Contact" H 2300 1150 50  0000 C CNN
-F 2 "" H 2300 1350 50  0001 C CNN
+F 2 "little_mobile_stm32f0:KEYSTONE_109-2_Battery_Contact" H 2300 1350 50  0001 C CNN
 F 3 "" H 2300 1350 50  0001 C CNN
 	1    2300 1350
@@
 F 0 "J3" H 2300 1850 50  0000 C CNN
 F 1 "BAT- Contact" H 2300 1550 50  0000 C CNN
-F 2 "" H 2300 1750 50  0001 C CNN
+F 2 "little_mobile_stm32f0:KEYSTONE_109-2_Battery_Contact" H 2300 1750 50  0001 C CNN
 F 3 "" H 2300 1750 50  0001 C CNN
 	1    2300 1750
@@
 F 0 "J4" H 6100 2150 50  0000 C CNN
 F 1 "Header_SWD" H 6100 1750 50  0000 C CNN
-F 2 "Pin_Headers:Pin_Header_Angled_1x03_Pitch2.54mm" H 6100 1950 50  0001 C CNN
+F 2 "Pin_Headers:Pin_Header_Straight_1x03_Pitch2.54mm" H 6100 1950 50  0001 C CNN
 F 3 "" H 6100 1950 50  0001 C CNN
 	1    6100 1950
@@
 F 0 "J1" H 600 1450 50  0000 L CNN
 F 1 "USB_OTG" H 600 1350 50  0000 L CNN
-F 2 "" H 950 950 50  0001 C CNN
+F 2 "little_mobile_stm32f0:Molex_1050170001_MicroUSB_B" H 950 950 50  0001 C CNN
 F 3 "" H 950 950 50  0001 C CNN
 	1    800  1000
