File: _saved_little_mobile_stm32f0_micro.sch (KiCad schematic (older format))
At the start: 23 parts, among them SW1 SW_DIP_x01, SW2 SW_DIP_x01, U5 STM32F072RBTx, Y1 Crystal_GND24, Y2 32.768k

Commit message: pcb Layout nearly completed
Parts:
- SW1, SW2: footprint (none) -> little_mobile_stm32f0:FSMSM_TE_Switch
- Y1: value Crystal_GND24 -> 8MHz; footprint (none) -> little_mobile_stm32f0:LFXTAL069277Reel_Crystal_8MHz
- Y2: footprint (none) -> little_mobile_stm32f0:CM7V-T1A_32.768kHz_Crystal
Other:
- note added: "USING: TE Connectivity: FSMSM"
Changed lines of the file:
@@
 F 0 "SW1" H 2250 3100 50  0000 C CNN
 F 1 "SW_DIP_x01" H 2250 2800 50  0000 C CNN
-F 2 "" H 2250 2950 50  0001 C CNN
+F 2 "little_mobile_stm32f0:FSMSM_TE_Switch" H 2250 2950 50  0001 C CNN
 F 3 "" H 2250 2950 50  0001 C CNN
 	1    2250 2950
@@
 Wire Wire Line
 	2850 1900 2850 2150
-Text Notes 2500 2200 2    60   ~ 0
+Text Notes 2550 2350 2    60   ~ 0
 Reset Button
 Text Notes 6750 1300 2    60   ~ 0
@@
 F 0 "SW2" H 11000 2650 50  0000 C CNN
 F 1 "SW_DIP_x01" H 11000 2350 50  0000 C CNN
-F 2 "" H 11000 2500 50  0001 C CNN
+F 2 "little_mobile_stm32f0:FSMSM_TE_Switch" H 11000 2500 50  0001 C CNN
 F 3 "" H 11000 2500 50  0001 C CNN
 	1    11000 2500
@@
 F 0 "Y2" H 2650 6600 50  0000 C CNN
 F 1 "32.768k" H 2650 6300 50  0000 C CNN
-F 2 "" H 2650 6450 50  0001 C CNN
+F 2 "little_mobile_stm32f0:CM7V-T1A_32.768kHz_Crystal" H 2650 6450 50  0001 C CNN
 F 3 "" H 2650 6450 50  0001 C CNN
 	1    2650 6450
@@
 P 900 4800
 F 0 "Y1" H 1025 5000 50  0000 L CNN
-F 1 "Crystal_GND24" H 1025 4925 50  0000 L CNN
-F 2 "" H 900 4800 50  0001 C CNN
+F 1 "8MHz" H 1025 4925 50  0000 L CNN
+F 2 "little_mobile_stm32f0:LFXTAL069277Reel_Crystal_8MHz" H 900 4800 50  0001 C CNN
 F 3 "" H 900 4800 50  0001 C CNN
 	1    900  4800
@@
 Text Notes 600  4100 0    60   ~ 0
 8MHz Main Frequency Crystal\n449-LFXTAL069277REEL\n20pF Load Capacitance
+Text Notes 2050 2850 2    60   ~ 0
+USING: TE Connectivity: FSMSM
+Text Notes 10900 2250 2    60   ~ 0
+USING: TE Connectivity: FSMSM
 $EndSCHEMATC
