File: _saved_little_mobile_stm32f0_power.sch (KiCad schematic (older format))
At the start: 32 parts, among them U1 bq24073, U2 CSD87313DMS, U3 bq29732, U4 TPS63050RMW

Commit message: pcb Layout nearly completed
Parts:
- U1: footprint (none) -> little_mobile_stm32f0:bq24073
- U2: footprint (none) -> little_mobile_stm32f0:csd87313DMS
- U3: footprint (none) -> little_mobile_stm32f0:WSON_bq2973
- U4: footprint (none) -> little_mobile_stm32f0:VQFN_tps6350
Changed lines of the file:
@@
 F 0 "U1" H 2700 -1400 60  0000 C CNN
 F 1 "bq24073" H 2700 1100 60  0000 C CNN
-F 2 "" H 2150 950 60  0001 C CNN
+F 2 "little_mobile_stm32f0:bq24073" H 2150 950 60  0001 C CNN
 F 3 "" H 2150 950 60  0001 C CNN
 	1    2150 950
@@
 F 0 "U3" H 4400 4050 60  0000 C CNN
 F 1 "bq29732" H 4350 4750 60  0000 C CNN
-F 2 "" H 4050 4600 60  0001 C CNN
+F 2 "little_mobile_stm32f0:WSON_bq2973" H 4050 4600 60  0001 C CNN
 F 3 "" H 4050 4600 60  0001 C CNN
 	1    4050 4600
@@
 F 0 "U2" H 3400 4650 60  0000 C CNN
 F 1 "CSD87313DMS" H 3400 5550 60  0000 C CNN
-F 2 "" H 2900 5400 60  0001 C CNN
+F 2 "little_mobile_stm32f0:csd87313DMS" H 2900 5400 60  0001 C CNN
 F 3 "" H 2900 5400 60  0001 C CNN
 	1    2900 5400
@@
 F 0 "U4" H 7250 -200 60  0000 C CNN
 F 1 "TPS63050RMW" H 7250 1300 60  0000 C CNN
-F 2 "" H 6800 1150 60  0001 C CNN
+F 2 "little_mobile_stm32f0:VQFN_tps6350" H 6800 1150 60  0001 C CNN
 F 3 "" H 6800 1150 60  0001 C CNN
 	1    6800 1150
