File: little_mobile_stm32f0.kicad_pcb (KiCad board)
At the start: 2 copper layers, 82 x 20 mm, 64 parts, among them J1 USB_OTG, J2 BAT+ Contact, J3 BAT- Contact, J4 Header_SWD, SW1 SW_DIP_x01, SW2 SW_DIP_x01, U1 bq24073, U2 CSD87313DMS, U3 bq29732, U4 TPS63050RMW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

Commit message: board would be ready for production
Parts:
- added J5: TEST_POWER_RAW, Measurement_Points:Measurement_Point_Round-SMD-Pad_Small, F.Cu at (108.0, 105.2)
- added J6: TEST_3v3, Measurement_Points:Measurement_Point_Round-SMD-Pad_Small, F.Cu at (124.6, 102.4)
- moved R17 86.5 mm to (129.4, 119.0), turned to 180 degrees
- moved R8 4.50 mm to (110.8, 105.8)
- moved C6 3.50 mm to (117.6, 101.5)
- moved C7 3.50 mm to (121.3, 103.0)
- moved C8 3.50 mm to (116.8, 106.0)
- moved C9 3.50 mm to (118.3, 106.0)
- moved L1 3.50 mm to (114.5, 105.2)
- moved R14 3.50 mm to (117.6, 103.8)
- moved R15 3.50 mm to (122.8, 103.0)
- moved R16 3.50 mm to (119.8, 103.0)
- moved U4 3.50 mm to (114.0, 102.5)
- moved C16 2.00 mm to (132.9, 104.6)
- moved C10 2.00 mm to (145.6, 116.7)
- moved C11 2.00 mm to (145.6, 111.2)
- moved C12 2.00 mm to (148.8, 111.2)
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Connections:
- net Net-(U5-Pad10) renamed /little_mobile_stm32f0_micro/PC2
- net Net-(U5-Pad11) renamed /little_mobile_stm32f0_micro/PC3
- net Net-(U5-Pad15) renamed /little_mobile_stm32f0_micro/PA1
- net Net-(U5-Pad16) renamed /little_mobile_stm32f0_micro/PA2
- net Net-(U5-Pad17) renamed /little_mobile_stm32f0_micro/PA3
- net Net-(U5-Pad2) renamed /little_mobile_stm32f0_micro/PC13
- net Net-(U5-Pad20) renamed /little_mobile_stm32f0_micro/PA4
- net Net-(U5-Pad21) renamed /little_mobile_stm32f0_micro/PA5
- net Net-(U5-Pad22) renamed /little_mobile_stm32f0_micro/PA6
- net Net-(U5-Pad23) renamed /little_mobile_stm32f0_micro/PA7
- net Net-(U5-Pad24) renamed /little_mobile_stm32f0_micro/PC4
- net Net-(U5-Pad25) renamed /little_mobile_stm32f0_micro/PC5
- net Net-(U5-Pad26) renamed /little_mobile_stm32f0_micro/PB0
- net Net-(U5-Pad27) renamed /little_mobile_stm32f0_micro/PB1
- net Net-(U5-Pad28) renamed /little_mobile_stm32f0_micro/PB2
- net Net-(U5-Pad29) renamed /little_mobile_stm32f0_micro/PB10
- net Net-(U5-Pad30) renamed /little_mobile_stm32f0_micro/PB11
- net Net-(U5-Pad33) renamed /little_mobile_stm32f0_micro/PB12
- net Net-(U5-Pad34) renamed /little_mobile_stm32f0_micro/PB13
- net Net-(U5-Pad35) renamed /little_mobile_stm32f0_micro/PB14
- net Net-(U5-Pad36) renamed /little_mobile_stm32f0_micro/PB15
- net Net-(U5-Pad37) renamed /little_mobile_stm32f0_micro/PC6
- net Net-(U5-Pad38) renamed /little_mobile_stm32f0_micro/PC7
- net Net-(U5-Pad39) renamed /little_mobile_stm32f0_micro/PC8
- net Net-(U5-Pad40) renamed /little_mobile_stm32f0_micro/PC9
- net Net-(U5-Pad41) renamed /little_mobile_stm32f0_micro/PA8
- net Net-(U5-Pad42) renamed /little_mobile_stm32f0_micro/PA9
- net Net-(U5-Pad43) renamed /little_mobile_stm32f0_micro/PA10
- net Net-(U5-Pad50) renamed /little_mobile_stm32f0_micro/PA15
- net Net-(U5-Pad51) renamed /little_mobile_stm32f0_micro/PC10
- net Net-(U5-Pad52) renamed /little_mobile_stm32f0_micro/PC11
- net Net-(U5-Pad53) renamed /little_mobile_stm32f0_micro/PC12
- net Net-(U5-Pad54) renamed /little_mobile_stm32f0_micro/PD2
- net Net-(U5-Pad55) renamed /little_mobile_stm32f0_micro/PB3
- net Net-(U5-Pad56) renamed /little_mobile_stm32f0_micro/PB4
- net Net-(U5-Pad57) renamed /little_mobile_stm32f0_micro/PB5
- net Net-(U5-Pad58) renamed /little_mobile_stm32f0_micro/PB6
- net Net-(U5-Pad59) renamed /little_mobile_stm32f0_micro/PB7
- net Net-(U5-Pad61) renamed /little_mobile_stm32f0_micro/PB8
- net Net-(U5-Pad62) renamed /little_mobile_stm32f0_micro/PB9
- net Net-(U5-Pad8) renamed /little_mobile_stm32f0_micro/PC0
- net Net-(U5-Pad9) renamed /little_mobile_stm32f0_micro/PC1
Routing:
- net GND: track 74.8 -> 241.7 mm
- net /little_mobile_stm32f0_power/BAT-: track 79.9 -> 84.9 mm
- net /little_mobile_stm32f0_micro/NRST: track 38.4 -> 43.1 mm
- net /little_mobile_stm32f0_power/POWER_RAW: track 16.8 -> 19.5 mm
- net (no net): track 2.43 -> 0.00 mm
- net /little_mobile_stm32f0_micro/USB_D+: track 29.3 -> 27.2 mm
- net Net-(R17-Pad1): track 0.00 -> 2.04 mm
- net /little_mobile_stm32f0_micro/USB_D-: track 29.3 -> 27.3 mm
- net Net-(L1-Pad2): track 0.00 -> 1.70 mm
- net /little_mobile_stm32f0_power/3v3: track 90.1 -> 91.5 mm
- net /little_mobile_stm32f0_micro/SWD_IO: track 18.4 -> 17.1 mm
- net /little_mobile_stm32f0_micro/SWD_CLK: track 18.1 -> 16.8 mm
- net /little_mobile_stm32f0_power/EN2: track 11.1 -> 10.6 mm
Other:
- board size 82 x 20 mm -> 80 x 20 mm
