File: little_mobile_stm32f0.sch (KiCad schematic (older format))
At the start: 5 parts, among them J1 USB_OTG, J2 BAT+ Contact, J3 BAT- Contact, J4 Header_SWD

Commit message: board would be ready for production
Parts:
- added J5: TEST_POWER_RAW, symbol TEST_1P
- added J6: TEST_3v3, symbol TEST_1P
- J1: footprint (none) -> little_mobile_stm32f0:Molex_1050170001_MicroUSB_B
- J2, J3: footprint (none) -> little_mobile_stm32f0:KEYSTONE_109-2_Battery_Contact
- J4: footprint Pin_Headers:Pin_Header_Angled_1x03_Pitch2.54mm -> Pin_Headers:Pin_Header_Straight_1x03_Pitch2.54mm
Connections:
- net little_mobile_stm32f0_micro/VDD: now also J6.1
- net little_mobile_stm32f0_power/POWER_RAW: now also J5.1
Changed lines of the file:
@@
 $EndSheet
 $Sheet
-S 6500 700  1750 2900
+S 6500 700  1700 5350
 U 5B7834FE
 F0 "little_mobile_stm32f0_micro" 60
@@
 F6 "SWD_CLK" I L 6500 1950 60
 F7 "NRST" I L 6500 2050 60
+F8 "PD2" I L 6500 2550 60
+F9 "PC0" I L 6500 2650 60
+F10 "PC1" I L 6500 2750 60
+F11 "PC6" I L 6500 2850 60
+F12 "PC2" I L 6500 2950 60
+F13 "PC3" I L 6500 3050 60
+F14 "PC4" I L 6500 3150 60
+F15 "PC5" I L 6500 3250 60
+F16 "PC7" I L 6500 3350 60
+F17 "PC8" I L 6500 3450 60
+F18 "PC9" I L 6500 3550 60
+F19 "PC10" I L 6500 3650 60
+F20 "PC11" I L 6500 3750 60
+F21 "PC12" I L 6500 3850 60
+F22 "PC13" I L 6500 3950 60
+F23 "PA1" I L 6500 4050 60
+F24 "PA2" I L 6500 4150 60
+F25 "PA3" I L 6500 4250 60
+F26 "PA4" I L 6500 4350 60
+F27 "PA5" I L 6500 4450 60
+F28 "PA6" I L 6500 4550 60
+F29 "PA7" I L 6500 4650 60
+F30 "PA8" I L 6500 4750 60
+F31 "PA9" I L 6500 4850 60
+F32 "PA10" I L 6500 4950 60
+F33 "PA15" I L 6500 5050 60
+F34 "PB0" I L 6500 5150 60
+F35 "PB1" I L 6500 5250 60
+F36 "PB2" I L 6500 5350 60
+F37 "PB3" I L 6500 5450 60
+F38 "PB4" I L 6500 5550 60
+F39 "PB5" I L 6500 5650 60
+F40 "PB6" I L 6500 5750 60
+F41 "PB7" I L 6500 5850 60
+F42 "PB8" I L 6500 5950 60
+F43 "PB9" I R 8200 5950 60
+F44 "PB10" I R 8200 5850 60
+F45 "PB11" I R 8200 5750 60
+F46 "PB12" I R 8200 5650 60
+F47 "PB13" I R 8200 5550 60
+F48 "PB14" I R 8200 5450 60
+F49 "PB15" I R 8200 5350 60
 $EndSheet
 $Comp
@@
 F 0 "J2" H 2300 1450 50  0000 C CNN
 F 1 "BAT+ Contact" H 2300 1150 50  0000 C CNN
-F 2 "" H 2300 1350 50  0001 C CNN
+F 2 "little_mobile_stm32f0:KEYSTONE_109-2_Battery_Contact" H 2300 1350 50  0001 C CNN
 F 3 "" H 2300 1350 50  0001 C CNN
 	1    2300 1350
@@
 F 0 "J3" H 2300 1850 50  0000 C CNN
 F 1 "BAT- Contact" H 2300 1550 50  0000 C CNN
-F 2 "" H 2300 1750 50  0001 C CNN
+F 2 "little_mobile_stm32f0:KEYSTONE_109-2_Battery_Contact" H 2300 1750 50  0001 C CNN
 F 3 "" H 2300 1750 50  0001 C CNN
 	1    2300 1750
@@
 F 0 "J4" H 6100 2150 50  0000 C CNN
 F 1 "Header_SWD" H 6100 1750 50  0000 C CNN
-F 2 "Pin_Headers:Pin_Header_Angled_1x03_Pitch2.54mm" H 6100 1950 50  0001 C CNN
+F 2 "Pin_Headers:Pin_Header_Straight_1x03_Pitch2.54mm" H 6100 1950 50  0001 C CNN
 F 3 "" H 6100 1950 50  0001 C CNN
 	1    6100 1950
@@
 F 0 "J1" H 600 1450 50  0000 L CNN
 F 1 "USB_OTG" H 600 1350 50  0000 L CNN
-F 2 "" H 950 950 50  0001 C CNN
+F 2 "little_mobile_stm32f0:Molex_1050170001_MicroUSB_B" H 950 950 50  0001 C CNN
 F 3 "" H 950 950 50  0001 C CNN
 	1    800  1000
@@
 Text Notes 1950 1100 0    60   ~ 0
 Using KEYSTONE 109-2 \nBattery Contact\nfor LiIon 18650
+$Comp
+L TEST_1P J6
+U 1 1 5B798658
+P 6200 900
+F 0 "J6" H 6200 1170 50  0000 C CNN
+F 1 "TEST_3v3" H 6200 1100 50  0000 C CNN
+F 2 "" H 6400 900 50  0001 C CNN
+F 3 "" H 6400 900 50  0001 C CNN
+	1    6200 900
+	-1   0    0    1
+$EndComp
+$Comp
+L TEST_1P J5
+U 1 1 5B79895C
+P 5450 950
+F 0 "J5" H 5450 1220 50  0000 C CNN
+F 1 "TEST_POWER_RAW" H 5450 1150 50  0000 C CNN
+F 2 "" H 5650 950 50  0001 C CNN
+F 3 "" H 5650 950 50  0001 C CNN
+	1    5450 950
+	0    1    1    0
+$EndComp
+Wire Wire Line
+	6200 900  6200 800
+Connection ~ 6200 800
+Wire Wire Line
+	5050 950  5450 950
 $EndSCHEMATC
