File: little_mobile_stm32f0_micro.sch (KiCad schematic (older format))
At the start: 23 parts, among them SW1 SW_DIP_x01, SW2 SW_DIP_x01, U5 STM32F072RBTx, Y1 Crystal_GND24, Y2 32.768k

Commit message: board would be ready for production
Parts:
- SW1, SW2: footprint (none) -> little_mobile_stm32f0:FSMSM_TE_Switch
- Y1: value Crystal_GND24 -> 8MHz; footprint (none) -> little_mobile_stm32f0:LFXTAL069277Reel_Crystal_8MHz
- Y2: footprint (none) -> little_mobile_stm32f0:CM7V-T1A_32.768kHz_Crystal
Connections:
- net PC2: now reaches U5.10 (PC2/ADC_IN12/I2S2_MCK/SPI2_MISO)
- net PC3: now reaches U5.11 (PC3/ADC_IN13/I2S2_SD/SPI2_MOSI)
- net PA1: now reaches U5.15 (ADC_IN1/COMP1_INP/TIM15_CH1N/TIM2_CH2/TSC_G1_IO2/USART2_DE/USART2_RTS/USART4_RX/PA1)
- net PA2: now reaches U5.16 (ADC_IN2/COMP2_INM/COMP2_OUT/SYS_WKUP4/TIM15_CH1/TIM2_CH3/TSC_G1_IO3/USART2_TX/PA2)
- net PA3: now reaches U5.17 (ADC_IN3/COMP2_INP/TIM15_CH2/TIM2_CH4/TSC_G1_IO4/USART2_RX/PA3)
- net PC13: now reaches U5.2 (PC13/RTC_OUT_ALARM/RTC_OUT_CALIB/RTC_TAMP1/RTC_TS/SYS_WKUP2)
- net PA4: now reaches U5.20 (ADC_IN4/COMP1_INM/COMP2_INM/DAC_OUT1/I2S1_WS/SPI1_NSS/TIM14_CH1/TSC_G2_IO1/USART2_CK/PA4)
- net PA5: now reaches U5.21 (ADC_IN5/CEC/COMP1_INM/COMP2_INM/DAC_OUT2/I2S1_CK/SPI1_SCK/TIM2_CH1/TIM2_ETR/TSC_G2_IO2/PA5)
- net PA6: now reaches U5.22 (ADC_IN6/COMP1_OUT/I2S1_MCK/SPI1_MISO/TIM16_CH1/TIM1_BKIN/TIM3_CH1/TSC_G2_IO3/USART3_CTS/PA6)
- net PA7: now reaches U5.23 (ADC_IN7/COMP2_OUT/I2S1_SD/SPI1_MOSI/TIM14_CH1/TIM17_CH1/TIM1_CH1N/TIM3_CH2/TSC_G2_IO4/PA7)
- net PC4: now reaches U5.24 (PC4/ADC_IN14/USART3_TX)
- net PC5: now reaches U5.25 (PC5/ADC_IN15/SYS_WKUP5/TSC_G3_IO1/USART3_RX)
- net PB0: now reaches U5.26 (ADC_IN8/TIM1_CH2N/TIM3_CH3/TSC_G3_IO2/USART3_CK/PB0)
- net PB1: now reaches U5.27 (ADC_IN9/TIM14_CH1/TIM1_CH3N/TIM3_CH4/TSC_G3_IO3/USART3_DE/USART3_RTS/PB1)
- net PB2: now reaches U5.28 (TSC_G3_IO4/PB2)
- net PB10: now reaches U5.29 (CEC/I2C2_SCL/I2S2_CK/SPI2_SCK/TIM2_CH3/TSC_SYNC/USART3_TX/PB10)
- net PB11: now reaches U5.30 (I2C2_SDA/TIM2_CH4/TSC_G6_IO1/USART3_RX/PB11)
- net PB12: now reaches U5.33 (I2S2_WS/SPI2_NSS/TIM15_BKIN/TIM1_BKIN/TSC_G6_IO2/USART3_CK/PB12)
- net PB13: now reaches U5.34 (I2C2_SCL/I2S2_CK/SPI2_SCK/TIM1_CH1N/TSC_G6_IO3/USART3_CTS/PB13)
- net PB14: now reaches U5.35 (I2C2_SDA/I2S2_MCK/SPI2_MISO/TIM15_CH1/TIM1_CH2N/TSC_G6_IO4/USART3_DE/USART3_RTS/PB14)
- net PB15: now reaches U5.36 (I2S2_SD/RTC_REFIN/SPI2_MOSI/SYS_WKUP7/TIM15_CH1N/TIM15_CH2/TIM1_CH3N/PB15)
- net PC6: now reaches U5.37 (PC6/TIM3_CH1)
- net PC7: now reaches U5.38 (PC7/TIM3_CH2)
- net PC8: now reaches U5.39 (PC8/TIM3_CH3)
- net PC9: now reaches U5.40 (PC9/DAC_EXTI9/TIM3_CH4)
- net PA8: now reaches U5.41 (CRS_SYNC/RCC_MCO/TIM1_CH1/USART1_CK/PA8)
- net PA9: now reaches U5.42 (DAC_EXTI9/TIM15_BKIN/TIM1_CH2/TSC_G4_IO1/USART1_TX/PA9)
- net PA10: now reaches U5.43 (TIM17_BKIN/TIM1_CH3/TSC_G4_IO2/USART1_RX/PA10)
- net PA15: now reaches U5.50 (I2S1_WS/SPI1_NSS/TIM2_CH1/TIM2_ETR/USART2_RX/USART4_DE/USART4_RTS/PA15)
- net PC10: now reaches U5.51 (PC10/USART3_TX/USART4_TX)
- net PC11: now reaches U5.52 (PC11/USART3_RX/USART4_RX)
- net PC12: now reaches U5.53 (PC12/USART3_CK/USART4_CK)
- net PD2: now reaches U5.54 (PD2/TIM3_ETR/USART3_DE/USART3_RTS)
- net PB3: now reaches U5.55 (I2S1_CK/SPI1_SCK/TIM2_CH2/TSC_G5_IO1/PB3)
- net PB4: now reaches U5.56 (I2S1_MCK/SPI1_MISO/TIM17_BKIN/TIM3_CH1/TSC_G5_IO2/PB4)
- net PB5: now reaches U5.57 (I2C1_SMBA/I2S1_SD/SPI1_MOSI/SYS_WKUP6/TIM16_BKIN/TIM3_CH2/PB5)
- net PB6: now reaches U5.58 (I2C1_SCL/TIM16_CH1N/TSC_G5_IO3/USART1_TX/PB6)
- net PB7: now reaches U5.59 (I2C1_SDA/TIM17_CH1N/TSC_G5_IO4/USART1_RX/USART4_CTS/PB7)
- net PB8: now reaches U5.61 (CAN_RX/CEC/I2C1_SCL/TIM16_CH1/TSC_SYNC/PB8)
- net PB9: now reaches U5.62 (CAN_TX/DAC_EXTI9/I2C1_SDA/I2S2_WS/IR_OUT/SPI2_NSS/TIM17_CH1/PB9)
- net PC0: now reaches U5.8 (PC0/ADC_IN10)
- net PC1: now reaches U5.9 (PC1/ADC_IN11)
Other:
- note added: "USING: TE Connectivity: FSMSM"
Changed lines of the file:
@@
 F 0 "SW1" H 2250 3100 50  0000 C CNN
 F 1 "SW_DIP_x01" H 2250 2800 50  0000 C CNN
-F 2 "" H 2250 2950 50  0001 C CNN
+F 2 "little_mobile_stm32f0:FSMSM_TE_Switch" H 2250 2950 50  0001 C CNN
 F 3 "" H 2250 2950 50  0001 C CNN
 	1    2250 2950
@@
 Wire Wire Line
 	2850 1900 2850 2150
-Text Notes 2500 2200 2    60   ~ 0
+Text Notes 2550 2350 2    60   ~ 0
 Reset Button
 Text Notes 6750 1300 2    60   ~ 0
@@
 F 0 "SW2" H 11000 2650 50  0000 C CNN
 F 1 "SW_DIP_x01" H 11000 2350 50  0000 C CNN
-F 2 "" H 11000 2500 50  0001 C CNN
+F 2 "little_mobile_stm32f0:FSMSM_TE_Switch" H 11000 2500 50  0001 C CNN
 F 3 "" H 11000 2500 50  0001 C CNN
 	1    11000 2500
@@
 F 0 "Y2" H 2650 6600 50  0000 C CNN
 F 1 "32.768k" H 2650 6300 50  0000 C CNN
-F 2 "" H 2650 6450 50  0001 C CNN
+F 2 "little_mobile_stm32f0:CM7V-T1A_32.768kHz_Crystal" H 2650 6450 50  0001 C CNN
 F 3 "" H 2650 6450 50  0001 C CNN
 	1    2650 6450
@@
 P 900 4800
 F 0 "Y1" H 1025 5000 50  0000 L CNN
-F 1 "Crystal_GND24" H 1025 4925 50  0000 L CNN
-F 2 "" H 900 4800 50  0001 C CNN
+F 1 "8MHz" H 1025 4925 50  0000 L CNN
+F 2 "little_mobile_stm32f0:LFXTAL069277Reel_Crystal_8MHz" H 900 4800 50  0001 C CNN
 F 3 "" H 900 4800 50  0001 C CNN
 	1    900  4800
@@
 Text Notes 600  4100 0    60   ~ 0
 8MHz Main Frequency Crystal\n449-LFXTAL069277REEL\n20pF Load Capacitance
+Text Notes 2050 2850 2    60   ~ 0
+USING: TE Connectivity: FSMSM
+Text Notes 10900 2250 2    60   ~ 0
+USING: TE Connectivity: FSMSM
+Text HLabel 3250 4450 0    60   Input ~ 0
+PD2
+Text HLabel 3250 4650 0    60   Input ~ 0
+PC0
+Text HLabel 3250 4750 0    60   Input ~ 0
+PC1
+Text HLabel 3250 5250 0    60   Input ~ 0
+PC6
+Text HLabel 3250 4850 0    60   Input ~ 0
+PC2
+Text HLabel 3250 4950 0    60   Input ~ 0
+PC3
+Text HLabel 3250 5050 0    60   Input ~ 0
+PC4
+Text HLabel 3250 5150 0    60   Input ~ 0
+PC5
+Text HLabel 3250 5350 0    60   Input ~ 0
+PC7
+Text HLabel 3250 5450 0    60   Input ~ 0
+PC8
+Text HLabel 3250 5550 0    60   Input ~ 0
+PC9
+Text HLabel 3250 5650 0    60   Input ~ 0
+PC10
+Text HLabel 3250 5750 0    60   Input ~ 0
+PC11
+Text HLabel 3250 5850 0    60   Input ~ 0
+PC12
+Text HLabel 3250 5950 0    60   Input ~ 0
+PC13
+Text HLabel 9250 3050 2    60   Input ~ 0
+PA1
+Text HLabel 9250 3150 2    60   Input ~ 0
+PA2
+Text HLabel 9250 3250 2    60   Input ~ 0
+PA3
+Text HLabel 9250 3350 2    60   Input ~ 0
+PA4
+Text HLabel 9250 3450 2    60   Input ~ 0
+PA5
+Text HLabel 9250 3550 2    60   Input ~ 0
+PA6
+Text HLabel 9250 3650 2    60   Input ~ 0
+PA7
+Text HLabel 9250 3750 2    60   Input ~ 0
+PA8
+Text HLabel 9250 3850 2    60   Input ~ 0
+PA9
+Text HLabel 9250 3950 2    60   Input ~ 0
+PA10
+Text HLabel 9250 4450 2    60   Input ~ 0
+PA15
+Text HLabel 9250 4650 2    60   Input ~ 0
+PB0
+Text HLabel 9250 4750 2    60   Input ~ 0
+PB1
+Text HLabel 9250 4850 2    60   Input ~ 0
+PB2
+Text HLabel 9250 4950 2    60   Input ~ 0
+PB3
+Text HLabel 9250 5050 2    60   Input ~ 0
+PB4
+Text HLabel 9250 5150 2    60   Input ~ 0
+PB5
+Text HLabel 9250 5250 2    60   Input ~ 0
+PB6
+Text HLabel 9250 5350 2    60   Input ~ 0
+PB7
+Text HLabel 9250 5450 2    60   Input ~ 0
+PB8
+Text HLabel 9250 5550 2    60   Input ~ 0
+PB9
+Text HLabel 9250 5650 2    60   Input ~ 0
+PB10
+Text HLabel 9250 5750 2    60   Input ~ 0
+PB11
+Text HLabel 9250 5850 2    60   Input ~ 0
+PB12
+Text HLabel 9250 5950 2    60   Input ~ 0
+PB13
+Text HLabel 9250 6050 2    60   Input ~ 0
+PB14
+Text HLabel 9250 6150 2    60   Input ~ 0
+PB15
 $EndSCHEMATC
